Commit message: compatibility tags

File: franka_description/robots/panda.gazebo.xacro (robot description, xacro)
@@ -1,5 +1,5 @@
 <?xml version="1.0"?>
 <robot xmlns:xacro="http://www.ros.org/wiki/xacro">
-    <xacro:macro name="panda_gazebo" params="robot_name">
+    <xacro:macro name="panda_gazebo" params="robot_name:='panda' load_gripper:='true'">
         <!-- Link0 -->
         <gazebo reference="${robot_name}_link0">
@@ -62,4 +62,5 @@
             <mu2>0.2</mu2>
         </gazebo>
+	<xacro:if value="$(arg load_gripper)">
         <!-- LinkRightFinger -->
         <gazebo reference="${robot_name}_rightfinger">
@@ -74,4 +75,5 @@
             <mu2>0.2</mu2>
         </gazebo>
+	</xacro:if>
     </xacro:macro>
 </robot>

File: franka_description/robots/panda.transmission.xacro (robot description, xacro)
@@ -1,5 +1,5 @@
 <?xml version="1.0"?>
 <robot xmlns:xacro="http://www.ros.org/wiki/xacro">
-    <xacro:macro name="panda_transmission" params="robot_name">
+    <xacro:macro name="panda_transmission" params="robot_name:='panda' load_gripper:='true'">
         <!-- Load Gazebo lib and set the robot namespace -->
         <gazebo>
@@ -78,4 +78,5 @@
             </actuator>
         </transmission>
+	<xacro:if value="$(arg load_gripper)">
         <transmission name="${robot_name}_leftfinger">
             <type>transmission_interface/SimpleTransmission</type>
@@ -98,4 +99,5 @@
             </actuator>
         </transmission>
+        </xacro:if>
     </xacro:macro>
 </robot>

File: franka_description/robots/panda_arm.xacro (robot description, xacro)
@@ -10,10 +10,4 @@
     </xacro:unless>
     <!-- for simulation -->
-    <link name="world" />
-    <joint name="robot_to_world" type="fixed">
-      <parent link="world" />
-      <child link="${arm_id}_link0" />
-      <origin xyz="0.0 0.0 0.0" rpy="0.0 0.0 0.0" />
-    </joint>
     <xacro:property name="joint_damping" value="1.0"/>
     <!-- end for simulation -->
