Commit message: revised down the masses to make robot more responsive

File: franka_description/robots/panda_arm.xacro (robot description, xacro)
@@ -105,5 +105,5 @@
       <inertial>
         <origin xyz="0 0 0" rpy="0 0 0" />
-        <mass value="2.38" />
+        <mass value="1.38" />
         <inertia ixx="0.3" ixy="0.0" ixz="0.0" iyy="0.3" iyz="0.0" izz="0.3" />
       </inertial>
@@ -135,5 +135,5 @@
       <inertial>
         <origin xyz="0 0 0" rpy="0 0 0" />
-        <mass value="2.43" />
+        <mass value="0.43" />
         <inertia ixx="0.3" ixy="0.0" ixz="0.0" iyy="0.3" iyz="0.0" izz="0.3" />
       </inertial>
@@ -165,5 +165,5 @@
       <inertial>
         <origin xyz="0 0 0" rpy="0 0 0" />
-        <mass value="3.5" />
+        <mass value="0.5" />
         <inertia ixx="0.3" ixy="0.0" ixz="0.0" iyy="0.3" iyz="0.0" izz="0.3" />
       </inertial>
@@ -195,5 +195,5 @@
       <inertial>
         <origin xyz="0 0 0" rpy="0 0 0" />
-        <mass value="1.47" />
+        <mass value="0.47" />
         <inertia ixx="0.3" ixy="0.0" ixz="0.0" iyy="0.3" iyz="0.0" izz="0.3" />
       </inertial>
