Commit message: Modify fingers collision and friction

File: franka_description/robots/hand.urdf.xacro (robot description, xacro)
@@ -3,3 +3,11 @@
   <xacro:include filename="hand.xacro"/>
   <xacro:hand ns="panda" safety_distance="0.03"/>
+  <xacro:macro name="hand_gazebo">
+ 	<gazebo reference="hand">
+    	<mu1>10000.0</mu1>
+  		<mu2>10000.0</mu2>
+  		<minDepth>0.003</minDepth>
+  		<maxVel>0</maxVel>
+	    <self_collide>true</self_collide>
+    </gazebo>
 </robot>

File: franka_description/robots/hand.xacro (robot description, xacro)
@@ -69,6 +69,16 @@
         <origin xyz="0 0.005 0.045" rpy="0 0 0"/>
         <geometry>
-          <sphere radius="${0.01+safety_distance}"  />
+          <box size="0.02 0.02 0.02"  />
         </geometry>
+        <surface>
+          <friction>
+           <ode>
+            <mu>10000.0</mu>
+            <mu2>10000.0</mu2>
+            <minDepth>0.003</minDepth>
+	    <maxVel>0</maxVel>
+           </ode>
+          </friction>
+       </surface>
       </collision>
       <!-- for simulation -->
@@ -90,6 +100,16 @@
         <origin xyz="0 -0.005 0.045" rpy="0 0 0"/>
         <geometry>
-          <sphere radius="${0.01+safety_distance}"  />
+          <box size="0.02 0.02 0.02"  />
         </geometry>
+        <surface>
+          <friction>
+           <ode>
+            <mu>10000.0</mu>
+            <mu2>10000.0</mu2>
+            <minDepth>0.003</minDepth>
+	    <maxVel>0</maxVel>
+           </ode>
+          </friction>
+       </surface>
       </collision>
       <!-- for simulation -->

Commit message: Minor fixes

File: franka_description/robots/hand.urdf.xacro (robot description, xacro)
@@ -3,11 +3,3 @@
   <xacro:include filename="hand.xacro"/>
   <xacro:hand ns="panda" safety_distance="0.03"/>
-  <xacro:macro name="hand_gazebo">
- 	<gazebo reference="hand">
-    	<mu1>10000.0</mu1>
-  		<mu2>10000.0</mu2>
-  		<minDepth>0.003</minDepth>
-  		<maxVel>0</maxVel>
-	    <self_collide>true</self_collide>
-    </gazebo>
 </robot>

File: franka_description/robots/hand.xacro (robot description, xacro)
@@ -71,14 +71,4 @@
           <box size="0.02 0.02 0.02"  />
         </geometry>
-        <surface>
-          <friction>
-           <ode>
-            <mu>10000.0</mu>
-            <mu2>10000.0</mu2>
-            <minDepth>0.003</minDepth>
-	    <maxVel>0</maxVel>
-           </ode>
-          </friction>
-       </surface>
       </collision>
       <!-- for simulation -->
@@ -102,14 +92,4 @@
           <box size="0.02 0.02 0.02"  />
         </geometry>
-        <surface>
-          <friction>
-           <ode>
-            <mu>10000.0</mu>
-            <mu2>10000.0</mu2>
-            <minDepth>0.003</minDepth>
-	    <maxVel>0</maxVel>
-           </ode>
-          </friction>
-       </surface>
       </collision>
       <!-- for simulation -->
