Commit message: added dummy inertial tags to links

File: franka_description/robots/hand.xacro (robot description, xacro)
@@ -10,4 +10,9 @@
     </xacro:unless>
     <link name="${ns}_hand">
+      <inertial>
+        <mass value="0.1"/>
+        <inertia ixx="1" ixy="0" ixz="0" iyy="1" iyz="0" izz="1" />
+        <origin/>
+      </inertial>
       <visual>
         <origin rpy="0 0 0" xyz="0 0 0"/>
@@ -27,4 +32,9 @@
     </link>
     <link name="${ns}_leftfinger">
+      <inertial>
+        <mass value="0.01"/>
+        <inertia ixx="1" ixy="0" ixz="0" iyy="1" iyz="0" izz="1" />
+        <origin/>
+      </inertial>
       <visual>
         <origin rpy="0 0 0" xyz="0 0 0"/>
@@ -43,4 +53,9 @@
     </link>
     <link name="${ns}_rightfinger">
+      <inertial>
+        <mass value="0.01"/>
+        <inertia ixx="1" ixy="0" ixz="0" iyy="1" iyz="0" izz="1" />
+        <origin/>
+      </inertial>
       <visual>
         <origin rpy="0 0 0" xyz="0 0 0"/>

File: franka_description/robots/panda_arm.xacro (robot description, xacro)
@@ -10,4 +10,9 @@
     </xacro:unless>
     <link name="${arm_id}_link0">
+      <inertial>
+        <mass value="5"/>
+        <inertia ixx="1" ixy="0" ixz="0" iyy="1" iyz="0" izz="1" />
+        <origin/>
+      </inertial>
       <visual>
         <origin rpy="0 0 0" xyz="0 0 0"/>
@@ -27,4 +32,9 @@
     </link>
     <link name="${arm_id}_link1">
+      <inertial>
+        <mass value="1"/>
+        <inertia ixx="1" ixy="0" ixz="0" iyy="1" iyz="0" izz="1" />
+        <origin/>
+      </inertial>
       <visual>
         <origin rpy="0 0 0" xyz="0 0 0"/>
@@ -52,4 +62,9 @@
     </joint>
     <link name="${arm_id}_link2">
+      <inertial>
+        <mass value="0.5"/>
+        <inertia ixx="1" ixy="0" ixz="0" iyy="1" iyz="0" izz="1" />
+        <origin/>
+      </inertial>
       <visual>
         <origin rpy="0 0 0" xyz="0 0 0"/>
@@ -77,4 +92,9 @@
     </joint>
     <link name="${arm_id}_link3">
+      <inertial>
+        <mass value="0.3"/>
+        <inertia ixx="1" ixy="0" ixz="0" iyy="1" iyz="0" izz="1" />
+        <origin/>
+      </inertial>
       <visual>
         <origin rpy="0 0 0" xyz="0 0 0"/>
@@ -102,4 +122,9 @@
     </joint>
     <link name="${arm_id}_link4">
+      <inertial>
+        <mass value="0.3"/>
+        <inertia ixx="1" ixy="0" ixz="0" iyy="1" iyz="0" izz="1" />
+        <origin/>
+      </inertial>
       <visual>
         <origin rpy="0 0 0" xyz="0 0 0"/>
@@ -127,4 +152,9 @@
     </joint>
     <link name="${arm_id}_link5">
+      <inertial>
+        <mass value="0.3"/>
+        <inertia ixx="1" ixy="0" ixz="0" iyy="1" iyz="0" izz="1" />
+        <origin/>
+      </inertial>
       <visual>
         <origin rpy="0 0 0" xyz="0 0 0"/>
@@ -152,4 +182,9 @@
     </joint>
     <link name="${arm_id}_link6">
+      <inertial>
+        <mass value="0.3"/>
+        <inertia ixx="1" ixy="0" ixz="0" iyy="1" iyz="0" izz="1" />
+        <origin/>
+      </inertial>
       <visual>
         <origin rpy="0 0 0" xyz="0 0 0"/>
@@ -177,4 +212,9 @@
     </joint>
     <link name="${arm_id}_link7">
+      <inertial>
+        <mass value="0.3"/>
+        <inertia ixx="1" ixy="0" ixz="0" iyy="1" iyz="0" izz="1" />
+        <origin/>
+      </inertial>
       <visual>
         <origin rpy="0 0 0" xyz="0 0 0"/>

Commit message: removed duplicate inertia tags

File: franka_description/robots/hand.xacro (robot description, xacro)
@@ -10,9 +10,4 @@
     </xacro:unless>
     <link name="${ns}_hand">
-      <inertial>
-        <mass value="0.1"/>
-        <inertia ixx="1" ixy="0" ixz="0" iyy="1" iyz="0" izz="1" />
-        <origin/>
-      </inertial>
       <visual>
         <geometry>
@@ -34,9 +29,4 @@
     </link>
     <link name="${ns}_leftfinger">
-      <inertial>
-        <mass value="0.01"/>
-        <inertia ixx="1" ixy="0" ixz="0" iyy="1" iyz="0" izz="1" />
-        <origin/>
-      </inertial>
       <visual>
         <geometry>
@@ -58,9 +48,4 @@
     </link>
     <link name="${ns}_rightfinger">
-      <inertial>
-        <mass value="0.01"/>
-        <inertia ixx="1" ixy="0" ixz="0" iyy="1" iyz="0" izz="1" />
-        <origin/>
-      </inertial>
       <visual>
         <origin xyz="0 0 0" rpy="0 0 ${pi}"/>

File: franka_description/robots/panda_arm.xacro (robot description, xacro)
@@ -13,9 +13,4 @@
     <!-- end for simulation -->
     <link name="${arm_id}_link0">
-      <inertial>
-        <mass value="5"/>
-        <inertia ixx="1" ixy="0" ixz="0" iyy="1" iyz="0" izz="1" />
-        <origin/>
-      </inertial>
       <visual>
         <geometry>
@@ -37,9 +32,4 @@
     </link>
     <link name="${arm_id}_link1">
-      <inertial>
-        <mass value="1"/>
-        <inertia ixx="1" ixy="0" ixz="0" iyy="1" iyz="0" izz="1" />
-        <origin/>
-      </inertial>
       <visual>
         <geometry>
@@ -72,9 +62,4 @@
     </joint>
     <link name="${arm_id}_link2">
-      <inertial>
-        <mass value="0.5"/>
-        <inertia ixx="1" ixy="0" ixz="0" iyy="1" iyz="0" izz="1" />
-        <origin/>
-      </inertial>
       <visual>
         <geometry>
@@ -107,9 +92,4 @@
     </joint>
     <link name="${arm_id}_link3">
-      <inertial>
-        <mass value="0.3"/>
-        <inertia ixx="1" ixy="0" ixz="0" iyy="1" iyz="0" izz="1" />
-        <origin/>
-      </inertial>
       <visual>
         <geometry>
@@ -142,9 +122,4 @@
     </joint>
     <link name="${arm_id}_link4">
-      <inertial>
-        <mass value="0.3"/>
-        <inertia ixx="1" ixy="0" ixz="0" iyy="1" iyz="0" izz="1" />
-        <origin/>
-      </inertial>
       <visual>
         <geometry>
@@ -177,9 +152,4 @@
     </joint>
     <link name="${arm_id}_link5">
-      <inertial>
-        <mass value="0.3"/>
-        <inertia ixx="1" ixy="0" ixz="0" iyy="1" iyz="0" izz="1" />
-        <origin/>
-      </inertial>
       <visual>
         <geometry>
@@ -212,9 +182,4 @@
     </joint>
     <link name="${arm_id}_link6">
-      <inertial>
-        <mass value="0.3"/>
-        <inertia ixx="1" ixy="0" ixz="0" iyy="1" iyz="0" izz="1" />
-        <origin/>
-      </inertial>
       <visual>
         <geometry>
@@ -247,9 +212,4 @@
     </joint>
     <link name="${arm_id}_link7">
-      <inertial>
-        <mass value="0.3"/>
-        <inertia ixx="1" ixy="0" ixz="0" iyy="1" iyz="0" izz="1" />
-        <origin/>
-      </inertial>
       <visual>
         <geometry>

Commit message: changed hand collision parameters

File: franka_description/robots/hand.xacro (robot description, xacro)
@@ -34,5 +34,5 @@
         </geometry>
       </collision>
-      <collision>
+      <!--      <collision>
         <origin xyz="0 0 0.1" rpy="0 ${pi/2} ${pi/2}"/>
         <geometry>
@@ -51,5 +51,5 @@
           <sphere radius="${0.02+safety_distance}"  />
         </geometry>
-      </collision>
+      </collision> -->
       <!-- for simulation -->
       <inertial>
@@ -66,4 +66,10 @@
         </geometry>
       </visual>
+      <collision>
+        <origin xyz="0 0.005 0.045" rpy="0 0 0"/>
+        <geometry>
+          <sphere radius="${0.01+safety_distance}"  />
+        </geometry>
+      </collision>
       <!-- for simulation -->
       <inertial>
@@ -81,4 +87,10 @@
         </geometry>
       </visual>
+      <collision>
+        <origin xyz="0 -0.005 0.045" rpy="0 0 0"/>
+        <geometry>
+          <sphere radius="${0.01+safety_distance}"  />
+        </geometry>
+      </collision>
       <!-- for simulation -->
       <inertial>

Commit message: full finger collision mesh

File: franka_description/robots/hand.xacro (robot description, xacro)
@@ -16,4 +16,5 @@
         </geometry>
       </visual>
+	<!--
       <collision>
         <origin xyz="0 0 0.04" rpy="0 ${pi/2} ${pi/2}"/>
@@ -34,4 +35,5 @@
         </geometry>
       </collision>
+	-->
       <!--      <collision>
         <origin xyz="0 0 0.1" rpy="0 ${pi/2} ${pi/2}"/>
@@ -67,8 +69,13 @@
       </visual>
       <collision>
+        <geometry>
+          <mesh filename="package://franka_description/meshes/visual/finger.dae"/>
+        </geometry>
+	<!-- old values
         <origin xyz="0 0.005 0.045" rpy="0 0 0"/>
         <geometry>
           <sphere radius="${0.01+safety_distance}"  />
-        </geometry>
+		</geometry>
+	-->
       </collision>
       <!-- for simulation -->
@@ -88,8 +95,14 @@
       </visual>
       <collision>
+        <origin xyz="0 0 0" rpy="0 0 ${pi}"/>
+        <geometry>
+          <mesh filename="package://franka_description/meshes/visual/finger.dae"/>
+        </geometry>
+	<!--
         <origin xyz="0 -0.005 0.045" rpy="0 0 0"/>
         <geometry>
           <sphere radius="${0.01+safety_distance}"  />
-        </geometry>
+		</geometry>
+	-->
       </collision>
       <!-- for simulation -->
@@ -106,5 +119,5 @@
       <origin xyz="0 0 0.0584" rpy="0 0 0"/>
       <axis xyz="0 1 0"/>
-      <limit effort="20" lower="0.0" upper="0.04" velocity="0.2"/>
+      <limit effort="2000" lower="0.0" upper="0.04" velocity="0.2"/>
     </joint>
     <joint name="${ns}_finger_joint2" type="prismatic">
@@ -113,5 +126,5 @@
       <origin xyz="0 0 0.0584" rpy="0 0 0"/>
       <axis xyz="0 -1 0"/>
-      <limit effort="20" lower="0.0" upper="0.04" velocity="0.2"/>
+      <limit effort="2000" lower="0.0" upper="0.04" velocity="0.2"/>
       <mimic joint="${ns}_finger_joint1" />
     </joint>

Commit message: Change finger collisions

File: franka_description/robots/hand.xacro (robot description, xacro)
@@ -67,7 +67,7 @@
       </visual>
       <collision>
-        <origin xyz="0 0.005 0.045" rpy="0 0 0"/>
+        <origin xyz="0 0.0075 0.0425" rpy="0 0 0"/>
         <geometry>
-          <box size="0.02 0.02 0.02"  />
+          <box size="0.02 0.025 0.025"  />
         </geometry>
       </collision>
@@ -88,7 +88,7 @@
       </visual>
       <collision>
-        <origin xyz="0 -0.005 0.045" rpy="0 0 0"/>
+        <origin xyz="0 -0.0075 0.0425" rpy="0 0 0"/>
         <geometry>
-          <box size="0.02 0.02 0.02"  />
+          <box size="0.02 0.025 0.025"  />
         </geometry>
       </collision>
